File: Kicad/controller/Game console.kicad_pcb (KiCad board)
At the start: 2 copper layers, 150 x 90.2 mm, 27 parts, among them SW1 LB, SW10 B, SW11 Menu, SW12 X, SW13 Y, SW14 View, SW15 LT, SW16 RT, SW2 RB, SW3 D Pad top, SW4 D Pad right, SW5 D Pad Left, SW6 A, SW7 D Pad bottom, SW8 Reset, SW9 Home, U1 MCP3008

Commit message: basic cad complete and new shoulder board created for rb, lb, rt and lt triggers
Parts:
- removed SW1: LB, easyeda2kicad:SW-TH_TC-1102N-C-DL-B
- removed SW15: LT, easyeda2kicad:SW-TH_TC-1102N-C-DL-B
- removed SW16: RT, easyeda2kicad:SW-TH_TC-1102N-C-DL-B
- removed SW2: RB, easyeda2kicad:SW-TH_TC-1102N-C-DL-B
- added J1: Left-T, Connector_JST:JST_XH_B3B-XH-A_1x03_P2.50mm_Vertical, F.Cu at (63.0, 36.0)
- added J2: Conn_01x03, Connector_JST:JST_XH_B3B-XH-A_1x03_P2.50mm_Vertical, F.Cu at (176.5, 36.0)
Connections:
- A1 pad 13: Net-(A1-AGND) -> unconnected-(A1-AGND-Pad33)
- A1 pad 18: Net-(A1-AGND) -> unconnected-(A1-AGND-Pad33)
- A1 pad 23: Net-(A1-AGND) -> unconnected-(A1-AGND-Pad33)
- A1 pad 28: Net-(A1-AGND) -> unconnected-(A1-AGND-Pad33)
- A1 pad 3: Net-(A1-AGND) -> unconnected-(A1-AGND-Pad33)
- A1 pad 33: Net-(A1-AGND) -> unconnected-(A1-AGND-Pad33)
- A1 pad 38: Net-(A1-AGND) -> unconnected-(A1-AGND-Pad33)
- A1 pad 8: Net-(A1-AGND) -> unconnected-(A1-AGND-Pad33)
- C1 pad 2: Net-(A1-AGND) -> unconnected-(A1-AGND-Pad33)
- C2 pad 2: Net-(A1-AGND) -> unconnected-(A1-AGND-Pad33)
- Left1 pad 1: Net-(A1-AGND) -> unconnected-(A1-AGND-Pad33)
- Left1 pad 10: Net-(A1-AGND) -> unconnected-(A1-AGND-Pad33)
- Left1 pad 6: Net-(A1-AGND) -> unconnected-(A1-AGND-Pad33)
- Left1 pad 7: Net-(A1-AGND) -> unconnected-(A1-AGND-Pad33)
- Left1 pad 8: Net-(A1-AGND) -> unconnected-(A1-AGND-Pad33)
- Left1 pad 9: Net-(A1-AGND) -> unconnected-(A1-AGND-Pad33)
- Left1 pad b: Net-(A1-AGND) -> unconnected-(A1-AGND-Pad33)
- Right1 pad 1: Net-(A1-AGND) -> unconnected-(A1-AGND-Pad33)
- Right1 pad 10: Net-(A1-AGND) -> unconnected-(A1-AGND-Pad33)
- Right1 pad 6: Net-(A1-AGND) -> unconnected-(A1-AGND-Pad33)
- Right1 pad 7: Net-(A1-AGND) -> unconnected-(A1-AGND-Pad33)
- Right1 pad 8: Net-(A1-AGND) -> unconnected-(A1-AGND-Pad33)
- Right1 pad 9: Net-(A1-AGND) -> unconnected-(A1-AGND-Pad33)
- Right1 pad b: Net-(A1-AGND) -> unconnected-(A1-AGND-Pad33)
- SW10 pad 2: Net-(A1-AGND) -> unconnected-(A1-AGND-Pad33)
- SW11 pad 2: Net-(A1-AGND) -> unconnected-(A1-AGND-Pad33)
- SW12 pad 2: Net-(A1-AGND) -> unconnected-(A1-AGND-Pad33)
- SW13 pad 2: Net-(A1-AGND) -> unconnected-(A1-AGND-Pad33)
- SW14 pad 2: Net-(A1-AGND) -> unconnected-(A1-AGND-Pad33)
- SW3 pad 2: Net-(A1-AGND) -> unconnected-(A1-AGND-Pad33)
- SW4 pad 2: Net-(A1-AGND) -> unconnected-(A1-AGND-Pad33)
- SW5 pad 2: Net-(A1-AGND) -> unconnected-(A1-AGND-Pad33)
- SW6 pad 2: Net-(A1-AGND) -> unconnected-(A1-AGND-Pad33)
- SW7 pad 2: Net-(A1-AGND) -> unconnected-(A1-AGND-Pad33)
- SW8 pad 2: Net-(A1-AGND) -> unconnected-(A1-AGND-Pad33)
- SW9 pad 2: Net-(A1-AGND) -> unconnected-(A1-AGND-Pad33)
- U1 pad 14: Net-(A1-AGND) -> unconnected-(A1-AGND-Pad33)
- U1 pad 9: Net-(A1-AGND) -> unconnected-(A1-AGND-Pad33)
Routing:
- net Net-(A1-AGND): track 753.8 -> 0.00 mm
- net unconnected-(A1-AGND-Pad33): track 0.00 -> 753.5 mm
- net Net-(A1-GPIO5): track 54.8 -> 119.3 mm, vias 1 -> 2
- net Net-(A1-GPIO3): track 46.4 -> 53.4 mm, vias 0 -> 1
- net Net-(A1-GPIO4): track 62.4 -> 58.2 mm, vias 1 -> 2
- net Net-(A1-GPIO6): track 77.9 -> 77.7 mm, vias 0 -> 3

Commit message: doing the layout for pcb so I can make the perfect pcb board
Parts:
- removed REF** (x4): MountingHole_3.2mm_M3, MountingHole:MountingHole_3.2mm_M3
- added C3: 47 µF, Capacitor_THT:CP_Radial_D5.0mm_P2.00mm, F.Cu at (172.1, 105.5)
- added D1: 1N4148, Diode_THT:D_DO-35_SOD27_P7.62mm_Horizontal, F.Cu at (203.2, 96.0)
- added D2: LED, LED_THT:LED_D3.0mm, F.Cu at (187.2, 108.6)
- added D3: 1N4148, Diode_THT:D_DO-35_SOD27_P7.62mm_Horizontal, F.Cu at (218.7, 111.0)
- added J3: Conn_01x02, Connector_JST:JST_PH_B2B-PH-K_1x02_P2.00mm_Vertical, F.Cu at (256.5, 120.0)
- added J4: Conn_01x02, Connector_JST:JST_PH_B2B-PH-K_1x02_P2.00mm_Vertical, F.Cu at (47.5, 112.5)
- added Q1: PN2222A, Package_TO_SOT_THT:TO-92_Inline, F.Cu at (202.7, 67.4)
- added Q2: PN2222A, Package_TO_SOT_THT:TO-92_Inline, F.Cu at (208.2, 67.4)
- added R1: 1000, Resistor_THT:R_Axial_DIN0207_L6.3mm_D2.5mm_P10.16mm_Horizontal, F.Cu at (179.2, 88.7)
- added R2: 330, Resistor_THT:R_Axial_DIN0207_L6.3mm_D2.5mm_P10.16mm_Horizontal, F.Cu at (179.2, 94.0)
- added R3: 1000, Resistor_THT:R_Axial_DIN0207_L6.3mm_D2.5mm_P10.16mm_Horizontal, F.Cu at (179.2, 99.0)
- A1, SW8: moved to F.Cu
- J1: value Left-T -> Conn_01x04; footprint Connector_JST:JST_XH_B3B-XH-A_1x03_P2.50mm_Vertical -> Connector_JST:JST_XH_B4B-XH-A_1x04_P2.50mm_Vertical
- J2: value Conn_01x03 -> Conn_01x04; footprint Connector_JST:JST_XH_B3B-XH-A_1x03_P2.50mm_Vertical -> Connector_JST:JST_XH_B4B-XH-A_1x04_P2.50mm_Vertical
- moved J1 148.2 mm to (210.5, 21.5)
- moved J2 123.1 mm to (54.0, 23.5)
- moved g** 102.7 mm to (247.5, 22.0)
- moved Right1 93.0 mm to (229.2, 44.0)
- moved SW11 74.6 mm to (175.5, 44.0)
- moved SW6 61.0 mm to (135.2, 15.8)
- moved C2 61.0 mm to (165.2, 108.3), turned to 0 degrees
- moved C1 51.8 mm to (165.2, 104.2)
- moved SW9 47.6 mm to (120.5, 12.0)
- moved SW14 47.2 mm to (187.0, 43.5)
- moved U1 46.5 mm to (154.0, 88.7), turned to 0 degrees
- moved SW12 39.1 mm to (145.5, 22.0)
- moved SW8 35.1 mm to (160.0, 42.0), turned to 0 degrees
- moved SW10 33.4 mm to (168.2, 27.8)
- moved SW13 32.7 mm to (185.5, 27.0)
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Connections:
- A1 pad 26: unconnected-(A1-GPIO20-Pad26) -> Net-(A1-GPIO20)
- A1 pad 27: unconnected-(A1-GPIO21-Pad27) -> Net-(A1-GPIO21)
- A1 pad 29: unconnected-(A1-GPIO22-Pad29) -> Net-(A1-GPIO22)
- A1 pad 40: unconnected-(A1-VBUS-Pad40) -> VBUS
- A1 pad 5: Net-(A1-GPIO3) -> unconnected-(A1-GPIO3-Pad5)
- A1 pad 7: Net-(A1-GPIO5) -> unconnected-(A1-GPIO5-Pad7)
- J1 pad 2: Net-(A1-GPIO6) -> Net-(A1-3V3)
- J1 pad 3: Net-(A1-GPIO5) -> Net-(A1-GPIO6)
- J2 pad 2: Net-(A1-GPIO4) -> Net-(A1-3V3)
- J2 pad 3: Net-(A1-GPIO3) -> Net-(A1-GPIO4)
- U1 pad 5: unconnected-(U1-CH4-Pad5) -> Net-(J1-Pin_4)
- U1 pad 6: unconnected-(U1-CH5-Pad6) -> Net-(J2-Pin_4)
Routing:
- net unconnected-(A1-AGND-Pad33): track 753.5 -> 0.00 mm
- net Net-(A1-3V3): track 248.9 -> 0.00 mm, vias 5 -> 0
- net Net-(A1-GPIO5): track 119.3 -> 0.00 mm, vias 2 -> 0
- net Net-(A1-GPIO12): track 108.6 -> 0.00 mm, vias 1 -> 0
- net Net-(U1-CH1): track 78.4 -> 0.00 mm, vias 1 -> 0
- net Net-(A1-GPIO6): track 77.7 -> 0.00 mm, vias 3 -> 0
- net Net-(A1-GPIO27_ADC1): track 76.1 -> 0.00 mm, vias 1 -> 0
- net Net-(A1-GPIO13): track 64.8 -> 0.00 mm, vias 2 -> 0
- net Net-(A1-GPIO18): track 62.8 -> 0.00 mm, vias 1 -> 0
- net Net-(U1-CH2): track 61.8 -> 0.00 mm
- net Net-(U1-CH0): track 61.3 -> 0.00 mm, vias 1 -> 0
- net Net-(A1-GPIO4): track 58.2 -> 0.00 mm, vias 2 -> 0
- net Net-(A1-GPIO17): track 56.9 -> 0.00 mm, vias 1 -> 0
- net Net-(A1-GPIO26_ADC0): track 55.2 -> 0.00 mm, vias 1 -> 0
- net Net-(A1-GPIO3): track 53.4 -> 0.00 mm, vias 1 -> 0
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Other:
- board size 150 x 90.2 mm -> 237.5 x 119 mm
